File: alice.sch (KiCad schematic (older format))
At the start: 138 parts, among them U1 ATMega32U4

Commit message: Starts tracing
Parts:
- removed U1: ATMega32U4, symbol 8Bit-MCU:ATMega32U4
- added C1, C2: 22p, Capacitor_SMD:C_0805_2012Metric_Pad1.15x1.40mm_HandSolder, symbol passives:C_nonpol
- added C3, C4, C5, C6: 0.1u, Capacitor_SMD:C_0805_2012Metric_Pad1.15x1.40mm_HandSolder, symbol passives:C_nonpol
- added C7: 4.7u, Capacitor_SMD:C_0805_2012Metric_Pad1.15x1.40mm_HandSolder, symbol passives:C_nonpol
- added C8: 1u, Capacitor_SMD:C_0805_2012Metric_Pad1.15x1.40mm_HandSolder, symbol passives:C_nonpol
- added R1, R4: 10k, Resistor_SMD:R_0805_2012Metric_Pad1.15x1.40mm_HandSolder, symbol keyboard_parts:R
- added R2, R3: 22, Resistor_SMD:R_0805_2012Metric_Pad1.15x1.40mm_HandSolder, symbol keyboard_parts:R
- added RSW1: SW_PUSH, Button_Switch_SMD:SW_SPST_TL3342, symbol keyboard_parts:SW_PUSH
- added U1: ATMEGA32U4, Package_DFN_QFN:QFN-44-1EP_7x7mm_P0.5mm_EP5.2x5.2mm, symbol keyboard_parts:ATMEGA32U4
- added USB1: USB_mini_micro_B, keyboard_parts:USB_miniB_hirose_5S8, symbol keyboard_parts:USB_mini_micro_B
- added X1: XTAL_GND, Crystal:Crystal_SMD_3225-4Pin_3.2x2.5mm, symbol keyboard_parts:XTAL_GND
- renumbered D_B2 to D_B1, D_B1 to D_B2, K_B2 to K_B1, K_B1 to K_B2
Connections:
- net labels added: COL0, COL1, COL10, COL11, COL12, COL13, COL14, COL15, COL2, COL3, COL4, COL5, COL6, COL7, COL8, COL9, GND, ROW0, ROW1, ROW2, ROW3, ROW4, VUSB
- net labels removed: col0, col1, col10, col11, col12, col13, col14, col15, col2, col3, col4, col5, col6, col7, col8, col9, row0, row1, row2, row3, row4
- wire segments 274 -> 345
- no-connect marks 0 -> 7
Other:
- moved on the sheet: D_0, D_1, D_10, D_11, D_12, D_13, D_2, D_3, D_4, D_5, D_6, D_7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
