File: alice.kicad_pcb (KiCad board)
At the start: 2 copper layers, 337.2 x 122.6 mm, 152 parts, among them SW1 SW_PUSH, U2 ATMEGA32U4, X2 XTAL_GND

Commit message: Starts tracing
Parts:
- removed C10, C11, C12, C13, C14, C9: 22pF, Capacitor_SMD:C_0805_2012Metric_Pad1.15x1.40mm_HandSolder
- removed R5, R6: 10k, Resistor_SMD:R_0805_2012Metric_Pad1.15x1.40mm_HandSolder
- removed R7, R8: 22u, Resistor_SMD:R_0805_2012Metric_Pad1.15x1.40mm_HandSolder
- removed SW1: SW_PUSH, Button_Switch_SMD:SW_SPST_TL3342
- removed U2: ATMEGA32U4, Package_QFP:TQFP-44_10x10mm_P0.8mm
- removed X2: XTAL_GND, Crystal:Crystal_SMD_5032-4Pin_5.0x3.2mm
- added C1: 22p, Capacitor_SMD:C_0805_2012Metric_Pad1.15x1.40mm_HandSolder, B.Cu at (300.7, 199.1)
- added C2: 22p, Capacitor_SMD:C_0805_2012Metric_Pad1.15x1.40mm_HandSolder, B.Cu at (293.6, 199.1)
- added C3: 0.1u, Capacitor_SMD:C_0805_2012Metric_Pad1.15x1.40mm_HandSolder, B.Cu at (303.8, 173.2)
- added C4: 0.1u, Capacitor_SMD:C_0805_2012Metric_Pad1.15x1.40mm_HandSolder, B.Cu at (303.8, 171.2)
- added C5: 0.1u, Capacitor_SMD:C_0805_2012Metric_Pad1.15x1.40mm_HandSolder, B.Cu at (303.8, 169.2)
- added C6: 0.1u, Capacitor_SMD:C_0805_2012Metric_Pad1.15x1.40mm_HandSolder, B.Cu at (303.8, 167.1)
- added C7: 4.7u, Capacitor_SMD:C_0805_2012Metric_Pad1.15x1.40mm_HandSolder, B.Cu at (303.8, 165.1)
- added R1: 10k, Resistor_SMD:R_0805_2012Metric_Pad1.15x1.40mm_HandSolder, B.Cu at (317.0, 156.0)
- added R2: 22, Resistor_SMD:R_0805_2012Metric_Pad1.15x1.40mm_HandSolder, B.Cu at (297.2, 160.0)
- added R3: 22, Resistor_SMD:R_0805_2012Metric_Pad1.15x1.40mm_HandSolder, B.Cu at (299.2, 160.0)
- added R4: 10k, Resistor_SMD:R_0805_2012Metric_Pad1.15x1.40mm_HandSolder, B.Cu at (290.3, 216.7)
- added RSW1: SW_PUSH, Button_Switch_SMD:SW_SPST_TL3342, B.Cu at (323.1, 157.0)
- added U1: ATMEGA32U4, Package_DFN_QFN:QFN-44-1EP_7x7mm_P0.5mm_EP5.2x5.2mm, B.Cu at (294.6, 210.3)
- added X1: XTAL_GND, Crystal:Crystal_SMD_3225-4Pin_3.2x2.5mm, B.Cu at (297.2, 199.1)
- C8: value 22pF -> 1u
- K_SHIFT2_2: footprint keyswitches:Kailh_socket_optional -> keyswitches:Kailh_socket
- moved C8 129.0 mm to (291.3, 199.1), turned to 90 degrees
- moved USB1 22.6 mm to (301.5, 147.3)
- moved D_CAPS_LOCK1 6.44 mm to (159.3, 195.6)
- moved D_CTRL2 6.14 mm to (445.5, 239.3)
- moved D_13 5.89 mm to (467.9, 221.5)
- moved D_ENTER1 5.85 mm to (436.4, 200.2)
- moved D_12 4.58 mm to (327.7, 251.5)
- moved D_PGDN1 4.33 mm to (135.9, 200.7)
- moved D_ALT1 4.13 mm to (210.8, 240.0)
- moved D_10 3.59 mm to (242.6, 242.6)
- moved D_BSLSH2 3.56 mm to (458.2, 167.1)
- moved D_7 2.90 mm to (309.9, 177.8)
- moved D_BACKSPACE1 2.46 mm to (420.1, 165.6)
- moved D_Y1 2.17 mm to (304.8, 197.1)
- moved D_H1 2.05 mm to (311.7, 213.1)
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- renumbered USB2 to USB1
Connections:
- net row0 renamed ROW0
- net row1 renamed ROW1
- net row2 renamed ROW2
- net row3 renamed ROW3
- net row4 renamed ROW4
- K_0 pad 1: col11 -> COL11
- K_1 pad 1: col2 -> COL2
- K_10 pad 1: col2 -> COL5
- K_10_2 pad 1: col2 -> COL5
- K_11 pad 1: col3 -> COL6
- K_11_2 pad 1: col3 -> COL6
- K_12 pad 1: col4 -> COL8
- K_13 pad 1: col13 -> COL15
- K_2 pad 1: col3 -> COL3
- K_3 pad 1: col4 -> COL4
- K_4 pad 1: col5 -> COL5
- K_5 pad 1: col6 -> COL6
- K_6 pad 1: col7 -> COL7
- K_7 pad 1: col8 -> COL8
- K_8 pad 1: col9 -> COL9
- K_9 pad 1: col10 -> COL10
- K_A1 pad 1: col2 -> COL2
- K_ALT1 pad 1: col1 -> COL2
- K_ALT2 pad 1: col5 -> COL9
- K_B1 pad 1: col6 -> COL6
- K_B2 pad 1: col5 -> COL7
- K_BACKSPACE1 pad 1: col14 -> COL14
- K_BACKSPACE2 pad 2: col14 -> COL14
- K_BSLSH1 pad 1: col14 -> COL15
- K_BSLSH2 pad 1: col15 -> COL15
- K_C1 pad 1: col3 -> COL4
- K_CAPS_LOCK1 pad 1: col1 -> COL1
- K_CAPS_LOCK1_2 pad 2: col1 -> COL1
- K_COMMA1 pad 1: col9 -> COL10
- K_CTRL1 pad 1: col0 -> COL1
- K_CTRL2 pad 1: col6 -> COL15
- K_D1 pad 1: col4 -> COL4
- K_DOT1 pad 1: col10 -> COL11
- K_E1 pad 1: col4 -> COL4
- K_ENTER1 pad 1: col13 -> COL14
- K_EQUAL1 pad 1: col13 -> COL13
- K_F1 pad 1: col5 -> COL5
- K_G1 pad 1: col6 -> COL6
- K_H1 pad 1: col7 -> COL8
- K_I1 pad 1: col9 -> COL10
- K_J1 pad 1: col8 -> COL9
- K_K1 pad 1: col9 -> COL10
- K_L1 pad 1: col10 -> COL11
- K_M1 pad 1: col8 -> COL9
- K_MINUS1 pad 1: col12 -> COL12
- K_N1 pad 1: col7 -> COL8
- K_O1 pad 1: col10 -> COL11
- K_P1 pad 1: col11 -> COL12
- K_PGDN1 pad 1: col0 -> COL0
- K_PGUP1 pad 1: col0 -> COL0
- K_PRSCR1 pad 1: col0 -> COL0
- K_Q1 pad 1: col2 -> COL2
- K_QUOTE1 pad 1: col12 -> COL13
- K_R1 pad 1: col5 -> COL5
- K_S1 pad 1: col3 -> COL3
- K_SEMIC1 pad 1: col11 -> COL12
- K_SHIFT1 pad 1: col0 -> COL1
- K_SHIFT2 pad 1: col12 -> COL14
- K_SHIFT2_2 pad 2: col12 -> COL14
- K_SLASH1 pad 1: col11 -> COL12
- K_T1 pad 1: col6 -> COL6
- K_TAB1 pad 1: col1 -> COL1
- K_U1 pad 1: col8 -> COL9
- K_V1 pad 1: col4 -> COL5
- K_W1 pad 1: col3 -> COL3
- K_X1 pad 1: col2 -> COL3
- K_Y1 pad 1: col7 -> COL8
- K_Z1 pad 1: col1 -> COL2
- K_[1 pad 1: col12 -> COL13
- K_]1 pad 1: col13 -> COL14
- K_`1 pad 1: col1 -> COL1
- USB1 pad 1: VCC -> VUSB
Routing:
- net COL15: track 0.00 -> 171.1 mm, vias 0 -> 1
- net COL14: track 0.00 -> 162.9 mm, vias 0 -> 1
- net COL0: track 0.00 -> 153.6 mm
- net COL13: track 0.00 -> 136.8 mm, vias 0 -> 1
- net COL1: track 0.00 -> 125.8 mm
- net COL12: track 0.00 -> 117.5 mm, vias 0 -> 1
- net COL11: track 0.00 -> 95.1 mm, vias 0 -> 1
- net COL2: track 0.00 -> 92.6 mm
- net COL10: track 0.00 -> 88.7 mm, vias 0 -> 1
- net COL3: track 0.00 -> 70.0 mm
- net COL9: track 0.00 -> 69.0 mm, vias 0 -> 1
- net COL4: track 0.00 -> 50.7 mm
- net COL8: track 0.00 -> 49.0 mm, vias 0 -> 1
- net COL5: track 0.00 -> 31.4 mm
- net COL7: track 0.00 -> 30.5 mm
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Other:
- outline, holes or cut-outs redrawn

Commit message: Main tracing complete
Parts:
- moved D_13 5.38 mm to (462.8, 223.3)
- moved C4 2.70 mm to (302.0, 173.2)
- moved C5 2.70 mm to (302.0, 171.2)
- moved C7 2.70 mm to (302.0, 167.1)
- moved C3 2.70 mm to (302.0, 175.3)
- moved C6 2.70 mm to (302.0, 169.2)
- moved D_H1 2.18 mm to (310.4, 214.9)
Routing:
- net ROW0: track 0.00 -> 365.9 mm, vias 0 -> 2
- net ROW4: track 0.00 -> 364.1 mm, vias 0 -> 2
- net ROW3: track 0.00 -> 351.8 mm, vias 0 -> 2
- net ROW2: track 0.00 -> 344.7 mm, vias 0 -> 4
- net ROW1: track 0.00 -> 339.8 mm
- net VUSB: track 0.00 -> 154.4 mm, vias 0 -> 8
- net COL6: track 15.7 -> 150.0 mm, vias 0 -> 8
- net COL5: track 31.4 -> 163.4 mm, vias 0 -> 7
- net COL9: track 69.0 -> 180.6 mm, vias 1 -> 8
- net COL2: track 92.6 -> 194.7 mm, vias 0 -> 7
- net COL15: track 171.1 -> 272.6 mm, vias 1 -> 0
- net COL14: track 162.9 -> 260.8 mm, vias 1 -> 4
- net COL8: track 49.0 -> 142.2 mm, vias 1 -> 8
- net COL1: track 125.8 -> 216.3 mm, vias 0 -> 8
- net Net-(R1-Pad1): track 0.00 -> 83.8 mm, vias 0 -> 2
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
Commit message: Finished tracing
Routing:
- net GND: track 15.8 -> 51.5 mm, vias 0 -> 8
- net ROW2: track 344.7 -> 346.7 mm
- net Net-(C8-Pad1): track 9.16 -> 10.6 mm
- added copper zone on B.Cu, net GND
- added copper zone on F.Cu, net GND

Commit message: Convert IC to TQFP
Parts:
- U1: footprint Package_DFN_QFN:QFN-44-1EP_7x7mm_P0.5mm_EP5.2x5.2mm -> SMD_ICs:TQFP44
- moved R4 11.8 mm to (294.1, 227.8)
- moved U1 2.87 mm to (296.7, 212.3)
Routing:
- net VUSB: track 154.4 -> 117.6 mm, vias 8 -> 3
- net GND: track 51.5 -> 34.3 mm, vias 8 -> 5
- net Net-(R4-Pad2): track 2.73 -> 12.6 mm, vias 0 -> 2
- net COL10: track 159.8 -> 153.3 mm
- net COL9: track 180.6 -> 174.4 mm
- net COL8: track 142.2 -> 136.3 mm
- net COL7: track 93.7 -> 88.7 mm
- net ROW2: track 346.7 -> 342.1 mm, vias 4 -> 2
- net COL3: track 146.0 -> 143.3 mm
- net COL2: track 194.8 -> 192.2 mm
- net COL4: track 118.4 -> 115.9 mm
- net COL1: track 216.5 -> 213.9 mm
- net COL6: track 150.0 -> 147.5 mm
- net COL0: track 214.2 -> 211.8 mm
- net COL5: track 163.4 -> 160.9 mm
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