File: _saved_mad-hatter.sch (KiCad schematic (older format))
At the start: 155 parts, among them J1 XM7D-0512, J2 AVR-ISP-6, U1 ATMEGA32U4, X1 16MHz

Commit message: Improvements
Changed lines of the file:
@@
 	4100 9200 4100 9250
 Wire Wire Line
-	3550 10750 3550 10650
+	3550 10750 3550 10700
 Wire Wire Line
-	3550 10650 3350 10650
+	3550 10700 3350 10700
 Wire Wire Line
-	3350 10650 3350 11150
+	3350 10700 3350 11150
 Wire Wire Line
 	3350 11150 3550 11150
