File: mad-hatter.kicad_pcb (KiCad board)
At the start: 2 copper layers, 337.2 x 122.6 mm, 160 parts, among them J1 USB_B_Mini, U1 ATMEGA32U4, X1 16MHz

Commit message: Small fixes
Parts:
- K_0, K_1, K_2, K_3, K_4, K_5, K_6, K_7, K_8, K_9, K_A1, K_ALT1, K_ALT2, K_B1, K_B2, K_BACKSPACE1, K_BACKSPACE2, K_BSLSH1, K_BSLSH2, K_C1, K_CAPS_LOCK1, K_CAPS_LOCK1_2, K_COMMA1, K_CTRL1, K_CTRL2, K_D1, K_DOT1, K_E1, K_ENTER1, K_EQUAL1, K_F1, K_FN1, K_G1, K_GUI1, K_GUI1_2, K_H1, K_I1, K_J1, K_K1, K_L1, K_M1, K_MINUS1, K_N1, K_O1, K_P1, K_PGDN1, K_PGUP1, K_PRSCR1, K_Q1, K_QUOTE1, K_R1, K_S1, K_SEMIC1, K_SHIFT1, K_SHIFT2, K_SHIFT2_2, K_SLASH1, K_SPC1, K_SPC1_2, K_SPC2, K_T1, K_TAB1, K_U1, K_V1, K_W1, K_X1, K_Y1, K_Z1, K_[1, K_]1, K_`1: footprint acheronKeyboardSwitches:MX100H -> acheronKeyboardSwitches:MX100
Routing:
- net COL14: track 267.3 -> 250.8 mm, vias 2 -> 0
- net COL1: track 234.3 -> 222.7 mm, vias 5 -> 0
- net COL0: track 225.7 -> 233.3 mm, vias 3 -> 0
- net Net-(D_SPC1-Pad2): track 13.4 -> 20.4 mm
- net COL3: track 130.5 -> 137.0 mm, vias 4 -> 0
- net Net-(D_SHIFT2-Pad2): track 17.5 -> 23.7 mm
- net COL10: track 161.4 -> 155.7 mm, vias 4 -> 0
- net COL7: track 103.4 -> 98.1 mm, vias 4 -> 0
- net COL8: track 141.5 -> 136.5 mm, vias 5 -> 0
- net COL6: track 107.9 -> 113.0 mm, vias 6 -> 0
- net Net-(D_CAPS_LOCK1-Pad2): track 13.8 -> 18.6 mm
- net COL5: track 131.8 -> 136.6 mm, vias 5 -> 0
- net Net-(D_GUI1-Pad2): track 11.7 -> 15.9 mm
- net Net-(D_N1-Pad2): track 5.79 -> 9.78 mm
- net COL12: track 190.3 -> 186.3 mm, vias 4 -> 0
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